File: Project/Schematics & PCB Design/LIL_Transmitter/LIL_Transmitter.kicad_pcb (KiCad board)
At the start: 2 copper layers, 75 x 52 mm, 14 parts, among them J1 OUTPUT, SW1 1825910-6, SW2 1825910-6, SW3 1825910-6, U1 QAM-TX2-433, U2 ESP8266

Commit message: Schematics & PCB Designs Updated
Connections:
- U2 pad 19: unconnected-(U2-RX-Pad19) -> /G
- U2 pad 21: /G -> unconnected-(U2-D7-Pad21)
- U2 pad 22: /Y -> unconnected-(U2-D6-Pad22)
- U2 pad 23: /G1 -> /DAT
- U2 pad 26: /Y1 -> /Y
- U2 pad 27: /R1 -> /R
- U2 pad 28: /DAT -> /Y1
- U2 pad 29: /R -> /R1
- U2 pad 30: unconnected-(U2-D0-Pad30) -> /G1
Routing:
- net /G1: track 38.0 -> 24.5 mm
- net /DAT: track 30.1 -> 43.2 mm
- net /G: track 56.6 -> 61.7 mm
- net /R: track 26.3 -> 21.8 mm
- net /Y: track 29.1 -> 25.2 mm, vias 1 -> 0
- net /Y1: track 35.5 -> 33.5 mm, vias 0 -> 1
- net Net-(R3-Pad2): track 18.2 -> 19.5 mm
- net VCC: track 118.7 -> 119.7 mm
- net Net-(R6-Pad2): track 19.7 -> 20.2 mm
- net Net-(R5-Pad1): track 8.82 -> 9.32 mm
- net /R1: track 37.9 -> 37.6 mm, vias 0 -> 1
