File: Project/Schematics & PCB Design/LIL_Transmitter/LIL_Transmitter.kicad_sch (KiCad schematic)
At the start: 13 parts, among them J1 OUTPUT, SW1 1825910-6, SW2 1825910-6, SW3 1825910-6, U1 QAM-TX2-433, U2 ESP8266

Commit message: Schematics & PCB Designs Updated
Connections:
- net DAT: now also U2.23 (D5); no longer U2.28 (D2)
- net G: now also U2.19 (RX); no longer U2.21 (D7)
- net G1: now also U2.30 (D0); no longer U2.23 (D5)
- net R: now also U2.27 (D3); no longer U2.29 (D1)
- net R1: now also U2.29 (D1); no longer U2.27 (D3)
- net Y: now also U2.26 (D4); no longer U2.22 (D6)
- net Y1: now also U2.28 (D2); no longer U2.26 (D4)
Changed lines of the file:
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@@
+	)
+	(no_connect
+		(at 140.97 63.5)
 	)
 	(no_connect
@@
 	)
 	(no_connect
-		(at 140.97 45.72)
-	)
-	(no_connect
 		(at 140.97 40.64)
 	)
@@
 	)
 	(no_connect
+		(at 140.97 60.96)
+	)
+	(no_connect
 		(at 105.41 73.66)
-	)
-	(no_connect
-		(at 140.97 71.12)
 	)
 	(wire
@@
 		)
 	)
-	(label "R1"
+	(label "Y1"
+		(at 140.97 50.8 0)
+		(effects
+			(font
+				(size 1.27 1.27)
+			)
+			(justify left bottom)
+		)
+	)
+	(label "R"
 		(at 140.97 53.34 0)
 		(effects
@@
 		)
 	)
-	(label "G1"
+	(label "G"
+		(at 140.97 71.12 0)
+		(effects
+			(font
+				(size 1.27 1.27)
+			)
+			(justify left bottom)
+		)
+	)
+	(label "R1"
+		(at 140.97 48.26 0)
+		(effects
+			(font
+				(size 1.27 1.27)
+			)
+			(justify left bottom)
+		)
+	)
+	(label "DAT"
 		(at 140.97 58.42 0)
-		(effects
-			(font
-				(size 1.27 1.27)
-			)
-			(justify left bottom)
-		)
-	)
-	(label "R"
-		(at 140.97 48.26 0)
 		(effects
 			(font
@@
 		)
 	)
-	(label "G"
-		(at 140.97 63.5 0)
+	(label "G1"
+		(at 140.97 45.72 0)
 		(effects
 			(font
@@
 		)
 	)
-	(label "DAT"
-		(at 140.97 50.8 0)
-		(effects
-			(font
-				(size 1.27 1.27)
-			)
-			(justify left bottom)
-		)
-	)
-	(label "Y1"
+	(label "Y"
 		(at 140.97 55.88 0)
 		(effects
@@
 		(effects
 			(font
-				(size 1.27 1.27)
-			)
-			(justify left bottom)
-		)
-	)
-	(label "Y"
-		(at 140.97 60.96 0)
-		(effects
-			(font
